Commit message: fix collision and inertia and add comments

File: urdf/ouster.urdf.xacro (robot description, xacro)
@@ -1,4 +1,4 @@
 <?xml version="1.0"?>
-<!-- Revolute-Revolute Manipulator -->
+<!-- Ouster OS1 Lidar Sensor -->
 <robot name="os1" xmlns:xacro="http://www.ros.org/wiki/xacro">
 <xacro:macro name="os1_lidar" params="parent *origin name:=os1_lidar">
@@ -15,15 +15,22 @@
         <mesh filename="package://rooster_description/urdf/meshes/os1_mesh.dae" />
       </geometry>
-      <!--material name="Grey"-->
-      <!--color rgba="0.6 0.6 0.6 0.8"/-->
-      <!--/material-->
     </visual>
     <inertial>
+      <!-- CoM taken from CAD assuming constant density and mass 0.479 (best approximation available to real mass) -->
+      <origin xyz="-0.03775e-3 -2.161e-7 31.329e-3" rpy="0 0 0" />
+      <!-- mass taken from Ouster datasheet -->
       <mass value="0.455" />
-      <inertia ixx="1.0" ixy="0.0" ixz="0.0" iyy="1.0" iyz="0.0"
-      izz="1.0" />
+      <!-- Inertia tensor from CAD assuming constant density and mass 0.479 (best approximation vailable to real mass) -->
+      <inertia ixx="3.545e-4" ixy="6.051e-10" ixz="-3.736e-7" iyy="3.554e-4" iyz="-2.919e-9" izz="3.627e-4" />
     </inertial>
+    <collision>
+      <origin xyz="0 0 0.03675"/>
+      <geometry>
+        <cylinder radius="0.04350" length="0.07350" />
+      </geometry>
+    </collision>
   </link>
   <joint name="ouster_sensor_to_lidar" type="fixed">
+    <!-- origin queried from device -->
     <origin xyz="0 0 0.03618" rpy="0 0 ${pi}" />
     <parent link="os1_sensor" />
@@ -32,4 +39,5 @@
   <link name="os1_lidar" />
   <joint name="ouster_sensor_to_imu" type="fixed">
+    <!-- origin queried from device -->
     <origin xyz="0.006253 -0.011775 0.007645" rpy="0 0 0" />
     <parent link="os1_sensor" />

Commit message: adding simulation arg, rooster mesh and inertia

File: urdf/ouster.urdf.xacro (robot description, xacro)
@@ -2,5 +2,6 @@
 <!-- Ouster OS1 Lidar Sensor -->
 <robot name="os1" xmlns:xacro="http://www.ros.org/wiki/xacro">
-<xacro:macro name="os1_lidar" params="parent *origin name:=os1_lidar">
+<xacro:arg name="simulation" default="false" />
+<xacro:macro name="os1_device" params="parent *origin name:=os1_lidar">
   <joint name="${parent}_to_ouster" type="fixed">
     <xacro:insert_block name="origin"/>
@@ -31,18 +32,21 @@
     </collision>
   </link>
-  <joint name="ouster_sensor_to_lidar" type="fixed">
-    <!-- origin queried from device -->
-    <origin xyz="0 0 0.03618" rpy="0 0 ${pi}" />
-    <parent link="os1_sensor" />
-    <child link="os1_lidar" />
-  </joint>
-  <link name="os1_lidar" />
-  <joint name="ouster_sensor_to_imu" type="fixed">
-    <!-- origin queried from device -->
-    <origin xyz="0.006253 -0.011775 0.007645" rpy="0 0 0" />
-    <parent link="os1_sensor" />
-    <child link="os1_imu" />
-  </joint>
-  <link name="os1_imu" />
+  <!-- if simulated sensor, produce extra frames as fixed -->
+  <xacro:if value="$(arg simulation)">
+    <joint name="ouster_sensor_to_lidar" type="fixed">
+      <!-- origin queried from device -->
+      <origin xyz="0 0 0.03618" rpy="0 0 ${pi}" />
+      <parent link="os1_sensor" />
+      <child link="os1_lidar" />
+    </joint>
+    <link name="os1_lidar" />
+    <joint name="ouster_sensor_to_imu" type="fixed">
+      <!-- origin queried from device -->
+      <origin xyz="0.006253 -0.011775 0.007645" rpy="0 0 0" />
+      <parent link="os1_sensor" />
+      <child link="os1_imu" />
+    </joint>
+    <link name="os1_imu" />
+  </xacro:if>
 </xacro:macro>
 </robot>

File: urdf/rooster.urdf.xacro (robot description, xacro)
@@ -4,25 +4,47 @@
   <xacro:include filename="$(find realsense2_description)/urdf/_d435.urdf.xacro" />
   <xacro:include filename="$(find rooster_description)/urdf/ouster.urdf.xacro" />
+  <xacro:arg name="simulation" default="false" />
   <link name="base" />
-  <link name="realsense_parent" />
+  <link name="base_inertia">
+    <visual>
+      <origin xyz="0 0 0" rpy="0 0 0" />
+      <geometry>
+        <mesh filename="package://rooster_description/urdf/meshes/rooster_mount_v1.dae" />
+      </geometry>
+    </visual>
+    <inertial>
+      <!-- CoM computed from CAD assuming material is ABS (density 1.052e-6 kg/mm^3)-->
+      <origin xyz="-12.256e-3 -0.092e-3 -29.959e-3" rpy="0 0 0" />
+      <mass value="0.212" />
+      <inertia ixx="3.541e-4" ixy="5.656e-6" ixz="-6.046e-5"
+      iyy="5.340e-4" iyz="-7.84e-6" izz="3.672e-4" />
+    </inertial>
+    <collision>
+      <origin xyz="0 0 0" rpy="0 0 0" />
+      <geometry>
+        <mesh filename="package://rooster_description/urdf/meshes/rooster_mount_v1.dae" />
+      </geometry>
+    </collision>
+  </link>
+  <joint name="base_to_inertia" type="fixed">
+    <parent link="base" />
+    <child link="base_inertia" />
+    <origin xyz="0 0 0" rpy="0 0 0" />
+  </joint>
   <!-- add OS1 Ouster Lidar sensor -->
-  <os1_lidar name="os1_lidar" parent="base">
+  <os1_device name="os1_sensor" parent="base">
     <origin xyz="0 0 0" rpy="0 0 0" />
-  </os1_lidar>
+    <xacro:arg name="simulation" default="$(arg simulation)" />
+  </os1_device>
   <!-- add RealSense D435i (the mesh is actually the non-IMU version -->
   <sensor_d435 name="realsense_d435" parent="realsense_parent">
     <origin xyz="0 0 0" rpy="0 0 0" />
-    <xacro:arg name="use_nominal_extrinsics" default="true" />
+    <xacro:arg name="use_nominal_extrinsics" default="$(arg simulation)" />
   </sensor_d435>
+  <link name="realsense_parent" />
   <joint name="base_to_realsense" type="fixed">
-    <origin xyz="0.15 0 -0.15" rpy="0 0 0" />
+    <origin xyz="43.7e-3 7.5e-3 -58.5e-3" rpy="0 0 0" />
     <parent link="base" />
     <child link="realsense_parent" />
   </joint>
-  <link name="basealt" />
-  <joint name="basealt_to_lidar" type="fixed" >
-	  <parent link="os1_sensor" />
-	  <child link="basealt"/>
-	  <origin xyz="-0.025 -0.045 -0.054" rpy="0 0 ${pi}" />
-  </joint>
 </robot>

Commit message: make the rooster standalone robot

File: urdf/ouster.urdf.xacro (robot description, xacro)
@@ -3,5 +3,5 @@
 <robot name="os1" xmlns:xacro="http://www.ros.org/wiki/xacro">
 <xacro:arg name="simulation" default="false" />
-<xacro:macro name="os1_device" params="parent *origin name:=os1_lidar">
+<xacro:macro name="os1_device" params="parent *origin name:=os1_lidar simulation:=false">
   <joint name="${parent}_to_ouster" type="fixed">
     <xacro:insert_block name="origin"/>
@@ -33,5 +33,5 @@
   </link>
   <!-- if simulated sensor, produce extra frames as fixed -->
-  <xacro:if value="$(arg simulation)">
+  <xacro:if value="${simulation}">
     <joint name="ouster_sensor_to_lidar" type="fixed">
       <!-- origin queried from device -->

File: urdf/rooster.urdf.xacro (robot description, xacro)
@@ -4,48 +4,57 @@
   <xacro:include filename="$(find realsense2_description)/urdf/_d435i.urdf.xacro" />
   <xacro:include filename="$(find rooster_description)/urdf/ouster.urdf.xacro" />
-  <!-- TODO make the xacro parametric against rooster version -->
-  <xacro:arg name="simulation" default="false" />
-  <link name="base" />
-  <link name="base_inertia">
-    <visual>
+  <xacro:macro name="rooster_device" params="parent:=base *origin simulation:=false">
+    <!-- TODO make the xacro parametric against rooster version -->
+    <link name="${parent}" />
+    <link name="base_mount">
+      <visual>
+        <origin xyz="0 0 0" rpy="0 0 0" />
+        <geometry>
+          <mesh filename="package://rooster_description/urdf/meshes/rooster_mount_v3.dae" />
+        </geometry>
+      </visual>
+      <inertial>
+        <!-- TODO Update inertia parameters -->
+        <origin xyz="-12.256e-3 -0.092e-3 -29.959e-3" rpy="0 0 0" />
+        <mass value="0.212" />
+        <inertia ixx="3.541e-4" ixy="5.656e-6" ixz="-6.046e-5"
+                 iyy="5.340e-4" iyz="-7.84e-6" izz="3.672e-4" />
+        </inertial>
+        <collision>
+	  <origin xyz="7e-3 0 ${77.25e-3/2}" rpy="0 0 0" />
+          <geometry>
+            <box size="133e-3 114e-3 77.25e-3" />
+          </geometry>
+        </collision>
+    </link>
+    <joint name="${parent}_to_mount" type="fixed">
+      <parent link="${parent}" />
+      <child link="base_mount" />
+      <xacro:insert_block name="origin" />
+    </joint>
+    <!-- add OS1 Ouster Lidar sensor -->
+    <os1_device name="os1_sensor" parent="base_mount" simulation="${simulation}">
+      <origin xyz="0 0 77.258e-3" rpy="0 0 ${-pi/4}" />
+    </os1_device>
+    <!-- add RealSense D435i (the mesh is actually the non-IMU version -->
+    <sensor_d435i name="camera" parent="realsense_parent" use_nominal_extrinsics="${simulation}">
       <origin xyz="0 0 0" rpy="0 0 0" />
-      <geometry>
-        <mesh filename="package://rooster_description/urdf/meshes/rooster_mount_v3.dae" />
-      </geometry>
-    </visual>
-    <inertial>
-      <!-- TODO Update inertia parameters -->
-      <origin xyz="-12.256e-3 -0.092e-3 -29.959e-3" rpy="0 0 0" />
-      <mass value="0.212" />
-      <inertia ixx="3.541e-4" ixy="5.656e-6" ixz="-6.046e-5"
-      iyy="5.340e-4" iyz="-7.84e-6" izz="3.672e-4" />
-    </inertial>
-    <collision>
-	    <origin xyz="7e-3 0 ${77.25e-3/2}" rpy="0 0 0" />
-      <geometry>
-	      <box size="133e-3 114e-3 77.25e-3" />
-      </geometry>
-    </collision>
-  </link>
-  <joint name="base_to_inertia" type="fixed">
-    <parent link="base" />
-    <child link="base_inertia" />
-    <origin xyz="0 0 0" rpy="0 0 0" />
-  </joint>
-  <!-- add OS1 Ouster Lidar sensor -->
-  <os1_device name="os1_sensor" parent="base">
-    <origin xyz="0 0 77.258e-3" rpy="0 0 ${-pi/4}" />
-    <xacro:arg name="simulation" default="$(arg simulation)" />
-  </os1_device>
-  <!-- add RealSense D435i (the mesh is actually the non-IMU version -->
-  <sensor_d435 parent="realsense_parent">
-    <origin xyz="0 0 0" rpy="0 0 0" />
-    <xacro:arg name="use_nominal_extrinsics" default="$(arg simulation)" />
-  </sensor_d435>
-  <link name="realsense_parent" />
-  <joint name="base_to_realsense" type="fixed">
-    <origin xyz="73.65e-3 7.5e-3 50.75e-3" rpy="0 0 0" />
-    <parent link="base" />
-    <child link="realsense_parent" />
-  </joint>
+    </sensor_d435i>
+    <link name="realsense_parent" />
+    <joint name="base_to_realsense" type="fixed">
+      <origin xyz="73.65e-3 7.5e-3 50.75e-3" rpy="0 0 0" />
+      <parent link="base_mount" />
+      <child link="realsense_parent" />
+    </joint>
+    <!-- the geometric center of the bottom screws is not
+         perfectly coincident with the base frame
+         (i.e., geometry center of device,
+         coincident with ouster center) -->
+    <link name="bottom_screws_center" />
+    <joint name="base_mount_to_bottom_screws_center" type="fixed">
+      <origin xyz="0 0.475e-3 0" rpy="0 0 0" />
+      <parent link="base_mount" />
+      <child link="bottom_screws_center" />
+    </joint>
+  </xacro:macro>
 </robot>

Commit message: update names according to new conventions

File: urdf/ouster.urdf.xacro (robot description, xacro)
@@ -11,14 +11,14 @@
    limitations under the License.
 -->
-<!-- Ouster OS1 Lidar Sensor -->
-<robot name="os1" xmlns:xacro="http://www.ros.org/wiki/xacro">
+<!-- Ouster OS Lidar Sensor -->
+<robot name="os" xmlns:xacro="http://www.ros.org/wiki/xacro">
 <xacro:arg name="simulation" default="false" />
-<xacro:macro name="os1_device" params="parent *origin name:=os1_lidar simulation:=false">
+<xacro:macro name="os_device" params="parent *origin name:=os1_lidar simulation:=false">
   <joint name="${parent}_to_ouster" type="fixed">
     <xacro:insert_block name="origin"/>
     <parent link="${parent}" />
-    <child link="os1_sensor" />
+    <child link="os_sensor" />
   </joint>
-  <link name="os1_sensor">
+  <link name="os_sensor">
     <visual>
       <origin xyz="0 0 0" rpy="${pi/2} 0 ${pi/2}" />
@@ -51,12 +51,12 @@
       <child link="os1_lidar" />
     </joint>
-    <link name="os1_lidar" />
+    <link name="os_lidar" />
     <joint name="ouster_sensor_to_imu" type="fixed">
       <!-- origin queried from device -->
       <origin xyz="0.006253 -0.011775 0.007645" rpy="0 0 0" />
-      <parent link="os1_sensor" />
-      <child link="os1_imu" />
+      <parent link="os_sensor" />
+      <child link="os_imu" />
     </joint>
-    <link name="os1_imu" />
+    <link name="os_imu" />
   </xacro:if>
 </xacro:macro>

File: urdf/rooster.urdf.xacro (robot description, xacro)
@@ -44,8 +44,8 @@
       <xacro:insert_block name="origin" />
     </joint>
-    <!-- add OS1 Ouster Lidar sensor -->
-    <xacro:os1_device name="os1_sensor" parent="base_mount" simulation="${simulation}">
+    <!-- add OS Ouster Lidar sensor -->
+    <xacro:os_device name="os1_sensor" parent="base_mount" simulation="${simulation}">
       <origin xyz="0 0 77.258e-3" rpy="0 0 ${-pi/4}" />
-    </xacro:os1_device>
+    </xacro:os_device>
     <!-- add RealSense D435i (the mesh is actually the non-IMU version -->
     <xacro:sensor_d435i name="camera" parent="realsense_parent" use_nominal_extrinsics="${simulation}">

Commit message: fix

File: urdf/ouster.urdf.xacro (robot description, xacro)
@@ -48,6 +48,6 @@
       <!-- origin queried from device -->
       <origin xyz="0 0 0.03618" rpy="0 0 ${pi}" />
-      <parent link="os1_sensor" />
-      <child link="os1_lidar" />
+      <parent link="os_sensor" />
+      <child link="os_lidar" />
     </joint>
     <link name="os_lidar" />

Commit message: fix lidar frames

File: urdf/ouster.urdf.xacro (robot description, xacro)
@@ -44,8 +44,9 @@
   </link>
   <!-- if simulated sensor, produce extra frames as fixed -->
+  <!-- real device publishes these frames directly -->
   <xacro:if value="${simulation}">
     <joint name="ouster_sensor_to_lidar" type="fixed">
       <!-- origin queried from device -->
-      <origin xyz="0 0 0.03618" rpy="0 0 ${pi}" />
+      <origin xyz="0.006253 -0.011775 0.007645" rpy="0 0 0" />
       <parent link="os_sensor" />
       <child link="os_lidar" />
