Commit message: fix view_urdf failing because of missing base link

File: urdf/rooster_standalone.urdf.xacro (robot description, xacro)
@@ -15,4 +15,5 @@
   <xacro:arg name="simulation" default="false" />
   <xacro:arg name="ground_camera" default="false" />
+  <link name="base"/>
   <xacro:rooster_device parent="base" simulation="$(arg simulation)" ground_camera="$(arg ground_camera)">
     <!-- this transform makes the robot base coincident with the front camera link -->
