Commit message: adding main xacro, ouster xacro, import realsense

File: urdf/rooster.urdf.xacro (robot description, xacro)
@@ -1,38 +1,28 @@
 <?xml version="1.0"?>
 <robot name="rooster" xmlns:xacro="http://www.ros.org/wiki/xacro">
-	<link name="base">
-	  <visual>
-		  <origin xyz="0 0 0.03675"/>
-	    <geometry>
-		    <cylinder radius="0.04350" length="0.07350" />
-	    </geometry>
-	         <material name="Grey">
-       <color rgba="0.6 0.6 0.6 0.8"/>
-     </material>
-	  </visual>
-        </link>
-	<joint name="base_to_ouster" type="fixed">
-		<origin xyz="0 0 0" rpy="0 0 0" />
-		<parent link="base" />
-		<child link="os1_sensor" />
-	</joint>
-	<link name="os1_sensor"/>
-	<joint name="ouster_sensor_to_lidar" type="fixed">
-		<origin xyz="0 0 0.03618" rpy="0 0 0" />
-		<parent link="os1_sensor" />
-		<child link="os1_lidar" />
-	</joint>
-	<link name="os1_lidar" />
-	<joint name="ouster_sensor_to_imu" type="fixed">
-		<origin xyz="0.006253 -0.011775 0.007645" rpy="0 0 0" />
-		<parent link="os1_sensor" />
-		<child link="os1_imu" />
-	</joint>
-	<link name="os1_imu" />
-	<link name="realsense_parent" />
-	<joint name="base_to_realsense" type="fixed">
-		<origin xyz="0 0 0" rpy="0 0 0" />
-		<parent link="base" />
-		<child link="realsense_parent" />
-	</joint>
+  <!-- include the RealSense d435 from official Intel's repository -->
+  <xacro:include filename="$(find realsense2_description)/urdf/_d435.urdf.xacro" />
+  <xacro:include filename="$(find rooster_description)/urdf/ouster.urdf.xacro" />
+  <link name="base" />
+  <link name="realsense_parent" />
+  <!-- add OS1 Ouster Lidar sensor -->
+  <os1_lidar name="os1_lidar" parent="base">
+    <origin xyz="0 0 0" rpy="0 0 0" />
+  </os1_lidar>
+  <!-- add RealSense D435i (the mesh is actually the non-IMU version -->
+  <sensor_d435 name="realsense_d435" parent="realsense_parent">
+    <origin xyz="0 0 0" rpy="0 0 0" />
+    <xacro:arg name="use_nominal_extrinsics" default="true" />
+  </sensor_d435>
+  <joint name="base_to_realsense" type="fixed">
+    <origin xyz="0.15 0 -0.15" rpy="0 0 0" />
+    <parent link="base" />
+    <child link="realsense_parent" />
+  </joint>
+  <link name="basealt" />
+  <joint name="basealt_to_lidar" type="fixed" >
+	  <parent link="os1_sensor" />
+	  <child link="basealt"/>
+	  <origin xyz="-0.025 -0.045 -0.054" rpy="0 0 ${pi}" />
+  </joint>
 </robot>

Commit message: update rooster to V3

File: urdf/rooster.urdf.xacro (robot description, xacro)
@@ -4,4 +4,5 @@
   <xacro:include filename="$(find realsense2_description)/urdf/_d435.urdf.xacro" />
   <xacro:include filename="$(find rooster_description)/urdf/ouster.urdf.xacro" />
+  <!-- TODO make the xacro parametric against rooster version -->
   <xacro:arg name="simulation" default="false" />
   <link name="base" />
@@ -10,9 +11,9 @@
       <origin xyz="0 0 0" rpy="0 0 0" />
       <geometry>
-        <mesh filename="package://rooster_description/urdf/meshes/rooster_mount_v1.dae" />
+        <mesh filename="package://rooster_description/urdf/meshes/rooster_mount_v3.dae" />
       </geometry>
     </visual>
     <inertial>
-      <!-- CoM computed from CAD assuming material is ABS (density 1.052e-6 kg/mm^3)-->
+      <!-- TODO Update inertia parameters -->
       <origin xyz="-12.256e-3 -0.092e-3 -29.959e-3" rpy="0 0 0" />
       <mass value="0.212" />
@@ -21,7 +22,7 @@
     </inertial>
     <collision>
-      <origin xyz="0 0 0" rpy="0 0 0" />
+	    <origin xyz="7e-3 0 ${77.25e-3/2}" rpy="0 0 0" />
       <geometry>
-        <mesh filename="package://rooster_description/urdf/meshes/rooster_mount_v1.dae" />
+	      <box size="133e-3 114e-3 77.25e-3" />
       </geometry>
     </collision>
@@ -34,5 +35,5 @@
   <!-- add OS1 Ouster Lidar sensor -->
   <os1_device name="os1_sensor" parent="base">
-    <origin xyz="0 0 0" rpy="0 0 0" />
+    <origin xyz="0 0 77.258e-3" rpy="0 0 ${-pi/4}" />
     <xacro:arg name="simulation" default="$(arg simulation)" />
   </os1_device>
@@ -44,5 +45,5 @@
   <link name="realsense_parent" />
   <joint name="base_to_realsense" type="fixed">
-    <origin xyz="43.7e-3 7.5e-3 -58.5e-3" rpy="0 0 0" />
+    <origin xyz="73.65e-3 7.5e-3 50.75e-3" rpy="0 0 0" />
     <parent link="base" />
     <child link="realsense_parent" />

Commit message: add extra frames from kalibr for calibration checking

File: urdf/rooster.urdf.xacro (robot description, xacro)
@@ -68,4 +68,26 @@
       <child link="bottom_screws_center" />
     </joint>
+<link name="cam0_kalibr"/>
+<joint name="imu_to_cam0_kalibr" type="fixed">
+  <origin xyz=" 0.0424927  0.0646684 -0.0184578" rpy="1.59163 -3.1276 2.36028" />
+  <parent link="os1_imu" />
+  <child link="cam0_kalibr" />
+</joint>
+<link name="imu_kalibr0"/>
+<joint name="cam0_to_imu_kalibr" type="fixed">
+  <origin xyz=" 0.0156275 -0.0198165 -0.0754414" rpy="  1.54147 -0.780804 0.0346379" />  <parent link="camera_infra1_optical_frame" />
+  <child link="imu_kalibr0" />
+</joint>
+<link name="cam1_kalibr"/>
+<joint name="imu_to_cam1_kalibr" type="fixed">
+  <origin xyz=" 0.0779608  0.0293712 -0.0177457" rpy="  1.5916 -3.12759  2.36187" />
+  <parent link="os1_imu" />
+  <child link="cam1_kalibr" />
+</joint>
+<link name="imu_kalibr1"/>
+<joint name="cam1_to_imu_kalibr" type="fixed">
+  <origin xyz="-0.0345365  -0.019802 -0.0753032" rpy="  1.54156 -0.779214 0.0345594" />  <parent link="camera_infra2_optical_frame" />
+  <child link="imu_kalibr1" />
+</joint>
   </xacro:macro>
 </robot>

Commit message: add 40 deg down shim & camera

File: urdf/rooster.urdf.xacro (robot description, xacro)
@@ -15,5 +15,5 @@
   <xacro:include filename="$(find realsense2_description)/urdf/_d435i.urdf.xacro" />
   <xacro:include filename="$(find rooster_description)/urdf/ouster.urdf.xacro" />
-  <xacro:macro name="rooster_device" params="parent:=base *origin simulation:=false">
+  <xacro:macro name="rooster_device" params="parent:=base *origin simulation:=false ground_camera:=false">
     <!-- TODO make the xacro parametric against rooster version -->
     <link name="${parent}" />
@@ -68,4 +68,28 @@
       <child link="bottom_screws_center" />
     </joint>
+    <xacro:if value="$(arg ground_camera)">
+      <link name="ground_camera_shim">
+        <visual>
+          <geometry>
+            <mesh filename="package://rooster_description/urdf/meshes/rooster_40deg_shim.dae" />
+          </geometry>
+        </visual>
+        <inertial>
+        <!-- TODO Update inertia parameters -->
+        <origin xyz="9.513e-3 -2.85e-3 -12.423e-3" rpy="0 0 0" />
+        <mass value="0.01" />
+        <inertia ixx="10.931e-6" ixy="0.177e-6" ixz="-0.253e-6"
+                 iyy="1.199e-6" iyz="0.075e-6" izz="10.21e-6" />
+        </inertial>
+      </link>
+      <joint name="ground_camera_shim_joint" type="fixed">
+        <origin xyz="59.5e-3 0 38.7e-3" rpy="0 0 0" />
+        <parent link="base_mount" />
+        <child link="ground_camera_shim" />
+      </joint>
+      <xacro:sensor_d435i name="ground_camera" parent="ground_camera_shim" use_nominal_extrinsics="${simulation}">
+        <origin xyz="14.345e-3 7.5e-3 -25.212e-3" rpy="0 ${pi*40.0/180.0} 0" />
+      </xacro:sensor_d435i>
+    </xacro:if>
   </xacro:macro>
 </robot>

File: urdf/rooster_standalone.urdf.xacro (robot description, xacro)
@@ -14,5 +14,6 @@
   <xacro:include filename="$(find rooster_description)/urdf/rooster.urdf.xacro" />
   <xacro:arg name="simulation" default="false" />
-  <xacro:rooster_device parent="base" simulation="$(arg simulation)">
+  <xacro:arg name="ground_camera" default="false" />
+  <xacro:rooster_device parent="base" simulation="$(arg simulation)" ground_camera="$(arg ground_camera)">
     <!-- this transform makes the robot base coincident with the front camera link -->
     <origin xyz="-0.08425 -0.025 -0.06325" rpy="0 0 0" />

Commit message: add even more checks

File: urdf/rooster.urdf.xacro (robot description, xacro)
@@ -76,5 +76,6 @@
 <link name="imu_kalibr0"/>
 <joint name="cam0_to_imu_kalibr" type="fixed">
-  <origin xyz=" 0.0156275 -0.0198165 -0.0754414" rpy="  1.54147 -0.780804 0.0346379" />  <parent link="camera_infra1_optical_frame" />
+  <origin xyz=" 0.0156275 -0.0198165 -0.0754414" rpy="  1.54147 -0.780804 0.0346379" />
+  <parent link="camera_infra1_optical_frame" />
   <child link="imu_kalibr0" />
 </joint>
@@ -87,6 +88,13 @@
 <link name="imu_kalibr1"/>
 <joint name="cam1_to_imu_kalibr" type="fixed">
-  <origin xyz="-0.0345365  -0.019802 -0.0753032" rpy="  1.54156 -0.779214 0.0345594" />  <parent link="camera_infra2_optical_frame" />
+  <origin xyz="-0.0345365  -0.019802 -0.0753032" rpy="  1.54156 -0.779214 0.0345594" />
+  <parent link="camera_infra2_optical_frame" />
   <child link="imu_kalibr1" />
+</joint>
+<link name="imu_kalibr0_gen2"/>
+<joint name="cam0_to_imu_kalibr_gen2" type="fixed" >
+  <origin xyz="0.0092806 -0.02235038 -0.07783546" rpy="1.5496029 -0.7735838 0.021965" />
+  <parent link="camera_infra1_optical_frame" />
+  <child link="imu_kalibr0_gen2" />
 </joint>
   </xacro:macro>

Commit message: remove bad link duplicating parent link, correct ground_camera substitution to xacro arg syntax

File: urdf/rooster.urdf.xacro (robot description, xacro)
@@ -17,5 +17,4 @@
   <xacro:macro name="rooster_device" params="parent:=base *origin simulation:=false ground_camera:=false">
     <!-- TODO make the xacro parametric against rooster version -->
-    <link name="${parent}" />
     <link name="base_mount">
       <visual>
@@ -68,5 +67,5 @@
       <child link="bottom_screws_center" />
     </joint>
-    <xacro:if value="$(arg ground_camera)">
+    <xacro:if value="${ground_camera}">
       <link name="ground_camera_shim">
         <visual>

Commit message: rename base_mount to rooster_base_mount to make it more obvious what base it is

File: urdf/rooster.urdf.xacro (robot description, xacro)
@@ -17,5 +17,5 @@
   <xacro:macro name="rooster_device" params="parent:=base *origin simulation:=false ground_camera:=false">
     <!-- TODO make the xacro parametric against rooster version -->
-    <link name="base_mount">
+    <link name="rooster_base_mount">
       <visual>
         <origin xyz="0 0 0" rpy="0 0 0" />
@@ -40,9 +40,9 @@
     <joint name="${parent}_to_mount" type="fixed">
       <parent link="${parent}" />
-      <child link="base_mount" />
+      <child link="rooster_base_mount" />
       <xacro:insert_block name="origin" />
     </joint>
     <!-- add OS Ouster Lidar sensor -->
-    <xacro:os_device name="os1_sensor" parent="base_mount" simulation="${simulation}">
+    <xacro:os_device name="os1_sensor" parent="rooster_base_mount" simulation="${simulation}">
       <origin xyz="0 0 77.258e-3" rpy="0 0 ${-pi/4}" />
     </xacro:os_device>
@@ -54,5 +54,5 @@
     <joint name="base_to_realsense" type="fixed">
       <origin xyz="73.65e-3 7.5e-3 50.75e-3" rpy="0 0 0" />
-      <parent link="base_mount" />
+      <parent link="rooster_base_mount" />
       <child link="realsense_parent" />
     </joint>
@@ -62,7 +62,7 @@
          coincident with ouster center) -->
     <link name="bottom_screws_center" />
-    <joint name="base_mount_to_bottom_screws_center" type="fixed">
+    <joint name="rooster_base_mount_to_bottom_screws_center" type="fixed">
       <origin xyz="0 0.475e-3 0" rpy="0 0 0" />
-      <parent link="base_mount" />
+      <parent link="rooster_base_mount" />
       <child link="bottom_screws_center" />
     </joint>
@@ -84,5 +84,5 @@
       <joint name="ground_camera_shim_joint" type="fixed">
         <origin xyz="59.5e-3 0 38.7e-3" rpy="0 0 0" />
-        <parent link="base_mount" />
+        <parent link="rooster_base_mount" />
         <child link="ground_camera_shim" />
       </joint>

Commit message: shorten rooster_base_mount to just rooster_mount

File: urdf/rooster.urdf.xacro (robot description, xacro)
@@ -17,5 +17,5 @@
   <xacro:macro name="rooster_device" params="parent:=base *origin simulation:=false ground_camera:=false">
     <!-- TODO make the xacro parametric against rooster version -->
-    <link name="rooster_base_mount">
+    <link name="rooster_mount">
       <visual>
         <origin xyz="0 0 0" rpy="0 0 0" />
@@ -40,9 +40,9 @@
     <joint name="${parent}_to_mount" type="fixed">
       <parent link="${parent}" />
-      <child link="rooster_base_mount" />
+      <child link="rooster_mount" />
       <xacro:insert_block name="origin" />
     </joint>
     <!-- add OS Ouster Lidar sensor -->
-    <xacro:os_device name="os1_sensor" parent="rooster_base_mount" simulation="${simulation}">
+    <xacro:os_device name="os1_sensor" parent="rooster_mount" simulation="${simulation}">
       <origin xyz="0 0 77.258e-3" rpy="0 0 ${-pi/4}" />
     </xacro:os_device>
@@ -54,5 +54,5 @@
     <joint name="base_to_realsense" type="fixed">
       <origin xyz="73.65e-3 7.5e-3 50.75e-3" rpy="0 0 0" />
-      <parent link="rooster_base_mount" />
+      <parent link="rooster_mount" />
       <child link="realsense_parent" />
     </joint>
@@ -62,7 +62,7 @@
          coincident with ouster center) -->
     <link name="bottom_screws_center" />
-    <joint name="rooster_base_mount_to_bottom_screws_center" type="fixed">
+    <joint name="rooster_mount_to_bottom_screws_center" type="fixed">
       <origin xyz="0 0.475e-3 0" rpy="0 0 0" />
-      <parent link="rooster_base_mount" />
+      <parent link="rooster_mount" />
       <child link="bottom_screws_center" />
     </joint>
@@ -84,5 +84,5 @@
       <joint name="ground_camera_shim_joint" type="fixed">
         <origin xyz="59.5e-3 0 38.7e-3" rpy="0 0 0" />
-        <parent link="rooster_base_mount" />
+        <parent link="rooster_mount" />
         <child link="ground_camera_shim" />
       </joint>

Commit message: Reorganize ouster simulation, add realsense

File: urdf/rooster.urdf.xacro (robot description, xacro)
@@ -15,5 +15,11 @@
   <xacro:include filename="$(find realsense2_description)/urdf/_d435i.urdf.xacro" />
   <xacro:include filename="$(find ouster_description)/urdf/ouster.urdf.xacro" />
-  <xacro:macro name="rooster_device" params="parent:=base *origin simulation:=false ground_camera:=false">
+  <xacro:macro name="rooster_device" params="parent:=base
+                                             *origin
+                                             simulation:=false
+                                             ground_camera:=false
+                                             ouster_vertical_angle:=45
+                                             ouster_beams:=64
+                                             ouster_hz:=10">
     <!-- TODO make the xacro parametric against rooster version -->
     <link name="rooster_mount">
@@ -92,7 +98,31 @@
     </xacro:if>
     <!-- Bring in simulation data for Gazebo. -->
-    <!-- <xacro:if value="${simulation}"> -->
-      <xacro:include filename="$(find rooster_description)/urdf/ouster.gazebo" />
-    <!-- </xacro:if> -->
+    <xacro:if value="${simulation}">
+      <!-- Simulated Ouster -->
+      <xacro:include filename="$(find rooster_description)/urdf/gazebo/ouster.gazebo"/>
+      <xacro:ouster_gazebo name="ouster" min_vertical_angle="${ouster_vertical_angle}"
+                                         max_vertical_angle="${-ouster_vertical_angle}"
+                                         hz="${ouster_hz}"
+                                         lasers="${ouster_beams}">
+        <origin xyz="0 0 0" rpy="0 0 0" />
+      </xacro:ouster_gazebo>
+      <!-- Simulated Realsense -->
+      <xacro:include filename="$(find rooster_description)/urdf/gazebo/realsense_d435.gazebo"/>
+      <!-- Add front camera -->
+      <xacro:realsense_d435_gazebo name="camera">
+        <origin xyz="0 0 0" rpy="0 0 0"/>
+      </xacro:realsense_d435_gazebo>
+      <!-- Add ground camera -->
+      <xacro:if value="${ground_camera}">
+        <xacro:realsense_d435_gazebo name="ground_camera">
+          <origin xyz="0 0 0" rpy="0 0 0"/>
+        </xacro:realsense_d435_gazebo>
+      </xacro:if>
+      <!-- Add ground truth -->
+      <xacro:include filename="$(find rooster_description)/urdf/gazebo/ground_truth.gazebo"/>
+      <xacro:ground_truth_gazebo parent="${parent}">
+        <origin xyz="0 0 0" rpy="0 0 0"/>
+      </xacro:ground_truth_gazebo>
+    </xacro:if>
   </xacro:macro>
 </robot>
