Commit message: rename all references from rooster to frontier

File: urdf/frontier.urdf.xacro (robot description, xacro)
@@ -11,9 +11,9 @@
    limitations under the License.
 -->
-<robot name="rooster" xmlns:xacro="http://www.ros.org/wiki/xacro">
+<robot name="frontier" xmlns:xacro="http://www.ros.org/wiki/xacro">
   <!-- include the RealSense d435 from official Intel's repository -->
   <xacro:include filename="$(find realsense2_description)/urdf/_d435i.urdf.xacro" />
   <xacro:include filename="$(find ouster_description)/urdf/ouster.urdf.xacro" />
-  <xacro:macro name="rooster_device" params="parent:=base
+  <xacro:macro name="frontier_device" params="parent:=base
                                              *origin
                                              simulation:=false
@@ -23,10 +23,10 @@
                                              ouster_hz:=10
                                              ouster_rotation:=${-pi/4}">
-    <!-- TODO make the xacro parametric against rooster version -->
-    <link name="rooster_mount">
+    <!-- TODO make the xacro parametric against frontier version -->
+    <link name="frontier_mount">
       <visual>
         <origin xyz="0 0 0" rpy="0 0 0" />
         <geometry>
-          <mesh filename="package://rooster_description/urdf/meshes/rooster_mount_v3.dae" />
+          <mesh filename="package://frontier_description/urdf/meshes/frontier_mount_v3.dae" />
         </geometry>
       </visual>
@@ -47,9 +47,9 @@
     <joint name="${parent}_to_mount" type="fixed">
       <parent link="${parent}" />
-      <child link="rooster_mount" />
+      <child link="frontier_mount" />
       <xacro:insert_block name="origin" />
     </joint>
     <!-- add OS Ouster Lidar sensor -->
-    <xacro:os_device name="os1_sensor" parent="rooster_mount" simulation="${simulation}">
+    <xacro:os_device name="os1_sensor" parent="frontier_mount" simulation="${simulation}">
       <origin xyz="0 0 77.258e-3" rpy="0 0 ${ouster_rotation}" />
     </xacro:os_device>
@@ -61,5 +61,5 @@
     <joint name="base_to_realsense" type="fixed">
       <origin xyz="73.65e-3 7.5e-3 50.75e-3" rpy="0 0 0" />
-      <parent link="rooster_mount" />
+      <parent link="frontier_mount" />
       <child link="realsense_parent" />
     </joint>
@@ -69,7 +69,7 @@
          coincident with ouster center) -->
     <link name="bottom_screws_center" />
-    <joint name="rooster_mount_to_bottom_screws_center" type="fixed">
+    <joint name="frontier_mount_to_bottom_screws_center" type="fixed">
       <origin xyz="0 0.475e-3 0" rpy="0 0 0" />
-      <parent link="rooster_mount" />
+      <parent link="frontier_mount" />
       <child link="bottom_screws_center" />
     </joint>
@@ -78,5 +78,5 @@
         <visual>
           <geometry>
-            <mesh filename="package://rooster_description/urdf/meshes/rooster_40deg_shim.dae" />
+            <mesh filename="package://frontier_description/urdf/meshes/frontier_40deg_shim.dae" />
           </geometry>
         </visual>
@@ -91,5 +91,5 @@
       <joint name="ground_camera_shim_joint" type="fixed">
         <origin xyz="59.5e-3 0 38.7e-3" rpy="0 0 0" />
-        <parent link="rooster_mount" />
+        <parent link="frontier_mount" />
         <child link="ground_camera_shim" />
       </joint>
@@ -101,5 +101,5 @@
     <xacro:if value="${simulation}">
       <!-- Simulated Ouster -->
-      <xacro:include filename="$(find rooster_description)/urdf/gazebo/ouster.gazebo"/>
+      <xacro:include filename="$(find frontier_description)/urdf/gazebo/ouster.gazebo"/>
       <xacro:ouster_gazebo name="ouster" min_vertical_angle="${ouster_vertical_angle}"
                                          max_vertical_angle="${-ouster_vertical_angle}"
@@ -109,5 +109,5 @@
       </xacro:ouster_gazebo>
       <!-- Simulated Realsense -->
-      <xacro:include filename="$(find rooster_description)/urdf/gazebo/realsense_d435.gazebo"/>
+      <xacro:include filename="$(find frontier_description)/urdf/gazebo/realsense_d435.gazebo"/>
       <!-- Add front camera -->
       <xacro:realsense_d435_gazebo name="camera">
@@ -121,5 +121,5 @@
       </xacro:if>
       <!-- Add ground truth -->
-      <xacro:include filename="$(find rooster_description)/urdf/gazebo/ground_truth.gazebo"/>
+      <xacro:include filename="$(find frontier_description)/urdf/gazebo/ground_truth.gazebo"/>
       <xacro:ground_truth_gazebo parent="${parent}">
         <origin xyz="0 0 0" rpy="0 0 0"/>

File: urdf/frontier_standalone.urdf.xacro (robot description, xacro)
@@ -10,7 +10,7 @@
    See the License for the specific language governing permissions and
    limitations under the License. -->
-<robot name="rooster" xmlns:xacro="http://www.ros.org/wiki/xacro">
+<robot name="frontier" xmlns:xacro="http://www.ros.org/wiki/xacro">
   <!-- include the RealSense d435 from official Intel's repository -->
-  <xacro:include filename="$(find rooster_description)/urdf/rooster.urdf.xacro" />
+  <xacro:include filename="$(find frontier_description)/urdf/frontier.urdf.xacro" />
   <xacro:arg name="simulation" default="false" />
   <xacro:arg name="ground_camera" default="false" />
@@ -18,7 +18,7 @@
   <xacro:arg name="ouster_rotation" default="'${-pi/4}'" />
   <link name="base"/>
-  <xacro:rooster_device parent="base" simulation="$(arg simulation)" ground_camera="$(arg ground_camera)" ouster_rotation="$(arg ouster_rotation)">
+  <xacro:frontier_device parent="base" simulation="$(arg simulation)" ground_camera="$(arg ground_camera)" ouster_rotation="$(arg ouster_rotation)">
     <!-- this transform makes the robot base coincident with the front camera link -->
     <origin xyz="-0.08425 -0.025 -0.06325" rpy="0 0 0" />
-  </xacro:rooster_device>
+  </xacro:frontier_device>
 </robot>

Commit message: WIP Add side/rear cameras to xacro.

File: urdf/frontier.urdf.xacro (robot description, xacro)
@@ -19,4 +19,7 @@
                                              simulation:=false
                                              ground_camera:=false
+                                             left_camera:=false
+                                             right_camera:=false
+                                             rear_camera:=false
                                              ouster_vertical_angle:=45
                                              ouster_beams:=64
@@ -55,13 +58,50 @@
     </xacro:os_device>
     <!-- add RealSense D435i (the mesh is actually the non-IMU version -->
+    <!-- Front camera -->
     <xacro:sensor_d435i name="camera" parent="realsense_parent" use_nominal_extrinsics="${simulation}">
       <origin xyz="0 0 0" rpy="0 0 0" />
     </xacro:sensor_d435i>
     <link name="realsense_parent" />
-    <joint name="base_to_realsense" type="fixed">
+    <joint name="mount_to_realsense" type="fixed">
       <origin xyz="73.65e-3 7.5e-3 50.75e-3" rpy="0 0 0" />
       <parent link="frontier_mount" />
       <child link="realsense_parent" />
     </joint>
+    <!-- Left camera -->
+    <xacro:if value="${left_camera}">
+      <xacro:sensor_d435i name="camera_left" parent="realsense_left_parent" use_nominal_extrinsics="${simulation}">
+        <origin xyz="0 0 0" rpy="0 0 0" />
+      </xacro:sensor_d435i>
+      <link name="realsense_left_parent" />
+      <joint name="mount_to_realsense_left" type="fixed">
+        <origin xyz="7.5e-3 -73.65e-3 50.75e-3" rpy="0 0 ${pi/2}" />
+        <parent link="frontier_mount" />
+        <child link="realsense_left_parent" />
+      </joint>
+    </xacro:if>
+    <!-- Right camera -->
+    <xacro:if value="${right_camera}">
+      <xacro:sensor_d435i name="camera_right" parent="realsense_right_parent" use_nominal_extrinsics="${simulation}">
+        <origin xyz="0 0 0" rpy="0 0 0" />
+      </xacro:sensor_d435i>
+      <link name="realsense_right_parent" />
+      <joint name="mount_to_realsense_right" type="fixed">
+        <origin xyz="-7.5e-3 73.65e-3 50.75e-3" rpy="0 0 ${pi}" />
+        <parent link="frontier_mount" />
+        <child link="realsense_right_parent" />
+      </joint>
+    </xacro:if>
+    <!-- Rear camera -->
+    <xacro:if value="${rear_camera}">
+      <xacro:sensor_d435i name="camera_rear" parent="realsense_rear_parent" use_nominal_extrinsics="${simulation}">
+        <origin xyz="0 0 0" rpy="0 0 0" />
+      </xacro:sensor_d435i>
+      <link name="realsense_rear_parent" />
+      <joint name="mount_to_realsense_rear" type="fixed">
+        <origin xyz="-73.65e-3 -7.5e-3 50.75e-3" rpy="0 0 ${-pi/2}" />
+        <parent link="frontier_mount" />
+        <child link="realsense_rear_parent" />
+      </joint>
+    </xacro:if>
     <!-- the geometric center of the bottom screws is not
          perfectly coincident with the base frame

File: urdf/frontier_standalone.urdf.xacro (robot description, xacro)
@@ -10,13 +10,22 @@
    See the License for the specific language governing permissions and
    limitations under the License. -->
-<robot name="frontier" xmlns:xacro="http://www.ros.org/wiki/xacro">
+<robot name="frontier"
+  xmlns:xacro="http://www.ros.org/wiki/xacro">
   <!-- include the RealSense d435 from official Intel's repository -->
   <xacro:include filename="$(find frontier_description)/urdf/frontier.urdf.xacro" />
   <xacro:arg name="simulation" default="false" />
   <xacro:arg name="ground_camera" default="false" />
+  <xacro:arg name="left_camera" default="false" />
+  <xacro:arg name="right_camera" default="false" />
+  <xacro:arg name="rear_camera" default="false" />
   <!-- Need to put the arithmetic computation into quotes because args must be strings -->
   <xacro:arg name="ouster_rotation" default="'${-pi/4}'" />
   <link name="base"/>
-  <xacro:frontier_device parent="base" simulation="$(arg simulation)" ground_camera="$(arg ground_camera)" ouster_rotation="$(arg ouster_rotation)">
+  <xacro:frontier_device parent="base" simulation="$(arg simulation)"
+                                        ground_camera="$(arg ground_camera)"
+                                        left_camera="$(arg left_camera)"
+                                        right_camera="$(arg right_camera)"
+                                        rear_camera="$(arg rear_camera)"
+                                        ouster_rotation="$(arg ouster_rotation)">
     <!-- this transform makes the robot base coincident with the front camera link -->
     <origin xyz="-0.08425 -0.025 -0.06325" rpy="0 0 0" />

Commit message: adjust the new cameras' pose in urdf
Now the left, right, rear cameras are pointing correctly. The detailed
translation is to be confirmed.

File: urdf/frontier.urdf.xacro (robot description, xacro)
@@ -75,5 +75,5 @@
       <link name="realsense_left_parent" />
       <joint name="mount_to_realsense_left" type="fixed">
-        <origin xyz="7.5e-3 -73.65e-3 50.75e-3" rpy="0 0 ${pi/2}" />
+        <origin xyz="0 67.65e-3 50.75e-3" rpy="0 0 ${pi/2}" />
         <parent link="frontier_mount" />
         <child link="realsense_left_parent" />
@@ -87,5 +87,5 @@
       <link name="realsense_right_parent" />
       <joint name="mount_to_realsense_right" type="fixed">
-        <origin xyz="-7.5e-3 73.65e-3 50.75e-3" rpy="0 0 ${pi}" />
+        <origin xyz="0 -67.65e-3 50.75e-3" rpy="0 0 ${-pi/2}" />
         <parent link="frontier_mount" />
         <child link="realsense_right_parent" />
@@ -99,5 +99,5 @@
       <link name="realsense_rear_parent" />
       <joint name="mount_to_realsense_rear" type="fixed">
-        <origin xyz="-73.65e-3 -7.5e-3 50.75e-3" rpy="0 0 ${-pi/2}" />
+        <origin xyz="-73.65e-3 -7.5e-3 50.75e-3" rpy="0 0 ${pi}" />
         <parent link="frontier_mount" />
         <child link="realsense_rear_parent" />

Commit message: add option to load hesai

File: urdf/frontier.urdf.xacro (robot description, xacro)
@@ -15,8 +15,10 @@
   <xacro:include filename="$(find realsense2_description)/urdf/_d435i.urdf.xacro" />
   <xacro:include filename="$(find ouster_description)/urdf/ouster.urdf.xacro" />
+  <xacro:include filename="$(find hesai_description)/urdf/hesai.urdf.xacro" />
   <xacro:macro name="frontier_device" params="parent:=base
                                              *origin
                                              simulation:=false
                                              ground_camera:=false
+                                             hesai:=true
                                              ouster_vertical_angle:=45
                                              ouster_beams:=64
@@ -50,8 +52,16 @@
       <xacro:insert_block name="origin" />
     </joint>
-    <!-- add OS Ouster Lidar sensor -->
-    <xacro:os_device name="os1_sensor" parent="frontier_mount" simulation="${simulation}">
-      <origin xyz="0 0 77.258e-3" rpy="0 0 ${ouster_rotation}" />
-    </xacro:os_device>
+    <xacro:unless value="${hesai}">
+      <!-- add OS Ouster Lidar sensor -->
+      <xacro:os_device name="os1_sensor" parent="frontier_mount" simulation="${simulation}">
+        <origin xyz="0 0 77.258e-3" rpy="0 0 ${ouster_rotation}" />
+      </xacro:os_device>
+    </xacro:unless>
+    <!-- if it's a model with Hesai PandarXT -->
+    <xacro:if value="${hesai}">
+      <xacro:hesai_device name="pandar" parent="frontier_mount" simulation="${simulation}">
+        <origin xyz="0 0 77.7e-3" rpy="0 0 0" />
+      </xacro:hesai_device>
+    </xacro:if>
     <!-- add RealSense D435i (the mesh is actually the non-IMU version -->
     <xacro:sensor_d435i name="camera" parent="realsense_parent" use_nominal_extrinsics="${simulation}">

Commit message: fix microstrain

File: urdf/frontier.urdf.xacro (robot description, xacro)
@@ -1,4 +1,4 @@
 <?xml version="1.0"?>
-<!-- Copyright 2020 University of Oxford
+<!-- Copyright 2020-2022 University of Oxford
    Licensed under the Apache License, Version 2.0 (the "License");
    you may not use this file except in compliance with the License.
@@ -61,5 +61,6 @@
     <xacro:if value="${hesai}">
       <xacro:hesai_device name="pandar" parent="frontier_mount" simulation="${simulation}">
-        <origin xyz="0 0 77.7e-3" rpy="0 0 0" />
+        <!-- 4 mm standoff present, not shown in model -->
+        <origin xyz="0 0 81.7e-3" rpy="0 0 0" />
       </xacro:hesai_device>
     </xacro:if>
@@ -73,4 +74,20 @@
       <parent link="frontier_mount" />
       <child link="realsense_parent" />
+    </joint>
+    <link name="microstrain_imu">
+      <visual>
+        <origin xyz="4.849e-3 0.0 -2.363e-3" rpy="0.0 0.0 0.0"/>
+        <geometry>
+          <box size="32.898e-3 24.384e-3 11.125e-3"/>
+        </geometry>
+          <material name="microstrain_gray">
+            <color rgba="0.27 0.27 0.27 1.0"/>
+          </material>
+      </visual>
+    </link>
+    <joint name="frontier_mount_to_microstrain_imu" type="fixed">
+      <origin xyz="40.42e-3 -34.58733e-3 62.5e-3" rpy="0.0 0.0 ${-pi}"/>
+      <parent link="frontier_mount"/>
+      <child link="microstrain_imu"/>
     </joint>
     <!-- the geometric center of the bottom screws is not

Commit message: remove ground camera and other old names

File: urdf/frontier.urdf.xacro (robot description, xacro)
@@ -19,9 +19,8 @@
                                              *origin
                                              simulation:=false
-                                             ground_camera:=false
                                              hesai:=true
-                                             ouster_vertical_angle:=45
-                                             ouster_beams:=64
-                                             ouster_hz:=10
+                                             lidar_fov:=45
+                                             lidar_beams:=64
+                                             lidar_hz:=10
                                              ouster_rotation:=${-pi/4}">
     <!-- TODO make the xacro parametric against frontier version -->
@@ -54,5 +53,5 @@
     <xacro:unless value="${hesai}">
       <!-- add OS Ouster Lidar sensor -->
-      <xacro:os_device name="os1_sensor" parent="frontier_mount" simulation="${simulation}">
+      <xacro:os_device name="os_sensor" parent="frontier_mount" simulation="${simulation}">
         <origin xyz="0 0 77.258e-3" rpy="0 0 ${ouster_rotation}" />
       </xacro:os_device>
@@ -65,5 +64,5 @@
       </xacro:hesai_device>
     </xacro:if>
-    <!-- add RealSense D435i (the mesh is actually the non-IMU version -->
+    <!-- add RealSense D435i (the mesh is actually the non-IMU version) -->
     <xacro:sensor_d435i name="camera" parent="realsense_parent" use_nominal_extrinsics="${simulation}">
       <origin xyz="0 0 0" rpy="0 0 0" />
@@ -94,5 +93,5 @@
          perfectly coincident with the base frame
          (i.e., geometry center of device,
-         coincident with ouster center) -->
+         coincident with lidar's rotation center) -->
     <link name="bottom_screws_center" />
     <joint name="frontier_mount_to_bottom_screws_center" type="fixed">
@@ -101,36 +100,12 @@
       <child link="bottom_screws_center" />
     </joint>
-    <xacro:if value="${ground_camera}">
-      <link name="ground_camera_shim">
-        <visual>
-          <geometry>
-            <mesh filename="package://frontier_description/urdf/meshes/frontier_40deg_shim.dae" />
-          </geometry>
-        </visual>
-        <inertial>
-        <!-- TODO Update inertia parameters -->
-        <origin xyz="9.513e-3 -2.85e-3 -12.423e-3" rpy="0 0 0" />
-        <mass value="0.01" />
-        <inertia ixx="10.931e-6" ixy="0.177e-6" ixz="-0.253e-6"
-                 iyy="1.199e-6" iyz="0.075e-6" izz="10.21e-6" />
-        </inertial>
-      </link>
-      <joint name="ground_camera_shim_joint" type="fixed">
-        <origin xyz="59.5e-3 0 38.7e-3" rpy="0 0 0" />
-        <parent link="frontier_mount" />
-        <child link="ground_camera_shim" />
-      </joint>
-      <xacro:sensor_d435i name="ground_camera" parent="ground_camera_shim" use_nominal_extrinsics="${simulation}">
-        <origin xyz="14.345e-3 7.5e-3 -25.212e-3" rpy="0 ${pi*40.0/180.0} 0" />
-      </xacro:sensor_d435i>
-    </xacro:if>
     <!-- Bring in simulation data for Gazebo. -->
     <xacro:if value="${simulation}">
       <!-- Simulated Ouster -->
       <xacro:include filename="$(find frontier_description)/urdf/gazebo/ouster.gazebo"/>
-      <xacro:ouster_gazebo name="ouster" min_vertical_angle="${ouster_vertical_angle}"
-                                         max_vertical_angle="${-ouster_vertical_angle}"
-                                         hz="${ouster_hz}"
-                                         lasers="${ouster_beams}">
+      <xacro:ouster_gazebo name="ouster" min_vertical_angle="${lidar_fov}"
+                                         max_vertical_angle="${-lidar_fov}"
+                                         hz="${lidar_hz}"
+                                         lasers="${lidar_beams}">
         <origin xyz="0 0 0" rpy="0 0 0" />
       </xacro:ouster_gazebo>
@@ -141,10 +116,4 @@
         <origin xyz="0 0 0" rpy="0 0 0"/>
       </xacro:realsense_d435_gazebo>
-      <!-- Add ground camera -->
-      <xacro:if value="${ground_camera}">
-        <xacro:realsense_d435_gazebo name="ground_camera">
-          <origin xyz="0 0 0" rpy="0 0 0"/>
-        </xacro:realsense_d435_gazebo>
-      </xacro:if>
       <!-- Add ground truth -->
       <xacro:include filename="$(find frontier_description)/urdf/gazebo/ground_truth.gazebo"/>

File: urdf/frontier_standalone.urdf.xacro (robot description, xacro)
@@ -14,9 +14,8 @@
   <xacro:include filename="$(find frontier_description)/urdf/frontier.urdf.xacro" />
   <xacro:arg name="simulation" default="false" />
-  <xacro:arg name="ground_camera" default="false" />
   <!-- Need to put the arithmetic computation into quotes because args must be strings -->
   <xacro:arg name="ouster_rotation" default="'${-pi/4}'" />
   <link name="base"/>
-  <xacro:frontier_device parent="base" simulation="$(arg simulation)" ground_camera="$(arg ground_camera)" ouster_rotation="$(arg ouster_rotation)">
+  <xacro:frontier_device parent="base" simulation="$(arg simulation)" ouster_rotation="$(arg ouster_rotation)">
     <!-- this transform makes the robot base coincident with the front camera link -->
     <origin xyz="-0.08425 -0.025 -0.06325" rpy="0 0 0" />

Commit message: add mesh for gx4_25 IMU

File: urdf/frontier.urdf.xacro (robot description, xacro)
@@ -74,9 +74,10 @@
       <child link="realsense_parent" />
     </joint>
+    <!-- add Microstrain IMU -->
     <link name="microstrain_imu">
       <visual>
         <origin xyz="4.849e-3 0.0 -2.363e-3" rpy="0.0 0.0 0.0"/>
         <geometry>
-          <box size="32.898e-3 24.384e-3 11.125e-3"/>
+          <mesh filename="package://frontier_description/urdf/meshes/3dm_gx4_25.dae"/>
         </geometry>
           <material name="microstrain_gray">

Commit message: move microstrains to dedicated file, load the 45 one into the xacro

File: urdf/frontier.urdf.xacro (robot description, xacro)
@@ -16,4 +16,5 @@
   <xacro:include filename="$(find ouster_description)/urdf/ouster.urdf.xacro" />
   <xacro:include filename="$(find hesai_description)/urdf/hesai.urdf.xacro" />
+  <xacro:include filename="$(find frontier_description)/urdf/microstrain.urdf.xacro" />
   <xacro:macro name="frontier_device" params="parent:=base
                                              *origin
@@ -27,5 +28,5 @@
     <link name="frontier_mount">
       <visual>
-        <origin xyz="0 0 0" rpy="0 0 0" />
+        <origin xyz="0.0 0.0 0.0" rpy="0.0 0.0 0.0" />
         <geometry>
           <mesh filename="package://frontier_description/urdf/meshes/frontier_mount_v3.dae" />
@@ -74,21 +75,11 @@
       <child link="realsense_parent" />
     </joint>
-    <!-- add Microstrain IMU -->
-    <link name="microstrain_imu">
-      <visual>
-        <origin xyz="4.849e-3 0.0 -2.363e-3" rpy="0.0 0.0 0.0"/>
-        <geometry>
-          <mesh filename="package://frontier_description/urdf/meshes/3dm_gx4_25.dae"/>
-        </geometry>
-          <material name="microstrain_gray">
-            <color rgba="0.27 0.27 0.27 1.0"/>
-          </material>
-      </visual>
-    </link>
-    <joint name="frontier_mount_to_microstrain_imu" type="fixed">
-      <origin xyz="40.42e-3 -34.58733e-3 62.5e-3" rpy="0.0 0.0 ${-pi}"/>
-      <parent link="frontier_mount"/>
-      <child link="microstrain_imu"/>
-    </joint>
+    <!-- Add the Microstrain 3DM-GX4-45 for now -->
+    <!-- TODO make the xacro parametric against the IMU model -->
+    <xacro:microstrain_gx4_45 parent="frontier_mount" simulation="${simulation}">
+      <!-- the origin is the same for both versions because it's in the -->
+      <!-- middle of the screw holes at the bottom -->
+      <origin xyz="34.047e-3 -34.58733e-3 65.7e-3" rpy="${pi} 0.0 0.0"/>
+    </xacro:microstrain_gx4_45>
     <!-- the geometric center of the bottom screws is not
          perfectly coincident with the base frame
