Commit message: create unique frontier device

File: urdf/frontier.urdf.xacro (robot description, xacro)
@@ -17,34 +17,77 @@
   <xacro:include filename="$(find hesai_description)/urdf/hesai.urdf.xacro" />
   <xacro:include filename="$(find frontier_description)/urdf/microstrain.urdf.xacro" />
+  <xacro:include filename="$(find alphasense_description)/urdf/alphasense.urdf.xacro" />
   <xacro:macro name="frontier_device" params="parent:=base
                                              *origin
                                              simulation:=false
-                                             hesai:=true
-                                             lidar_fov:=45
-                                             lidar_beams:=64
-                                             lidar_hz:=10
-                                             ouster_rotation:=${-pi/4}">
-    <!-- TODO make the xacro parametric against frontier version -->
-    <link name="frontier_mount">
-      <visual>
-        <origin xyz="0.0 0.0 0.0" rpy="0.0 0.0 0.0" />
-        <geometry>
-          <mesh filename="package://frontier_description/urdf/meshes/frontier_mount_v3.dae" />
-        </geometry>
-      </visual>
-      <inertial>
-        <!-- TODO Update inertia parameters -->
-        <origin xyz="-12.256e-3 -0.092e-3 -29.959e-3" rpy="0 0 0" />
-        <mass value="0.212" />
-        <inertia ixx="3.541e-4" ixy="5.656e-6" ixz="-6.046e-5"
-                 iyy="5.340e-4" iyz="-7.84e-6" izz="3.672e-4" />
-        </inertial>
-        <collision>
-	  <origin xyz="7e-3 0 ${77.25e-3/2}" rpy="0 0 0" />
+                                             use_ouster:=false
+                                             use_realsense:=false
+                                             rotate_ouster:=false
+                                             raise_lidar:=false">
+    <xacro:property name="lidar_hz" value="10" />
+    <xacro:if value="${use_realsense}">
+      <xacro:if value="${raise_lidar}">
+        <!-- 4 mm standoff present, not shown in model -->
+        <xacro:property name="lidar_z" value="81.7e-3"/>
+      </xacro:if>
+      <xacro:unless value="${raise_lidar}">
+        <xacro:property name="lidar_z" value="77.7e-3"/>
+      </xacro:unless>
+    </xacro:if>
+    <xacro:unless value="${use_realsense}">
+      <!-- lidar is 1 mm higher than in the previous version of the halo -->
+      <xacro:property name="lidar_z" value="91.683e-3"/>
+    </xacro:unless>
+    <!-- Assuming we are using Ouster OS1-64 -->
+    <xacro:if value="${use_ouster}">
+      <xacro:property name="lidar_fov" value="45" />
+      <xacro:property name="lidar_beams" value="64"/>
+    </xacro:if>
+    <!-- assuming we are using Hesai XT32 -->
+    <xacro:unless value="${use_ouster}">
+      <xacro:property name="lidar_fov" value="31" />
+      <xacro:property name="lidar_beams" value="32"/>
+    </xacro:unless>
+    <xacro:if value="${rotate_ouster}">
+      <xacro:property name="ouster_rotation" value="${-pi/4}"/>
+    </xacro:if>
+    <xacro:unless value="${rotate_ouster}">
+      <xacro:property name="ouster_rotation" value="0"/>
+    </xacro:unless>
+    <!-- Assuming we are using RealSense D435i -->
+    <xacro:if value="${use_realsense}">
+      <link name="frontier_mount">
+        <visual>
+          <origin xyz="0.0 0.0 0.0" rpy="0.0 0.0 0.0" />
           <geometry>
-            <box size="133e-3 114e-3 77.25e-3" />
+            <mesh filename="package://frontier_description/urdf/meshes/frontier_mount_v6_realsense.dae" />
           </geometry>
-        </collision>
-    </link>
+        </visual>
+        <inertial>
+          <!-- TODO Update inertia parameters -->
+          <origin xyz="-12.256e-3 -0.092e-3 -29.959e-3" rpy="0 0 0" />
+          <mass value="0.212" />
+          <inertia ixx="3.541e-4" ixy="5.656e-6" ixz="-6.046e-5"
+                   iyy="5.340e-4" iyz="-7.84e-6" izz="3.672e-4" />
+          </inertial>
+          <collision>
+	    <origin xyz="7e-3 0 ${77.25e-3/2}" rpy="0 0 0" />
+            <geometry>
+              <box size="133e-3 114e-3 77.25e-3" />
+            </geometry>
+          </collision>
+      </link>
+    </xacro:if>
+    <!-- Assuming we are using Alphasense Core Dev Kit -->
+    <xacro:unless value="${use_realsense}">
+      <link name="frontier_mount">
+        <visual>
+          <geometry>
+            <mesh filename="package://frontier_description/urdf/meshes/frontier_mount_v6.dae" />
+          </geometry>
+        </visual>
+        <!-- TODO add inertia params -->
+      </link>
+    </xacro:unless>
     <joint name="${parent}_to_mount" type="fixed">
       <parent link="${parent}" />
@@ -52,34 +95,45 @@
       <xacro:insert_block name="origin" />
     </joint>
-    <xacro:unless value="${hesai}">
+    <!-- Assuming we are using Ouster OS1-64 -->
+    <xacro:if value="${use_ouster}">
       <!-- add OS Ouster Lidar sensor -->
       <xacro:os_device name="os_sensor" parent="frontier_mount" simulation="${simulation}">
-        <origin xyz="0 0 77.258e-3" rpy="0 0 ${ouster_rotation}" />
+        <origin xyz="0 0 ${lidar_z}" rpy="0 0 ${ouster_rotation}" />
       </xacro:os_device>
+    </xacro:if>
+    <!-- assuming we are using Hesai XT32 -->
+    <xacro:unless value="${use_ouster}">
+      <xacro:hesai_device name="pandar" parent="frontier_mount" simulation="${simulation}">
+          <origin xyz="0 0 ${lidar_z}" rpy="0 0 0" />
+      </xacro:hesai_device>
+      <!-- Only add the Microstrain if the Hesai XT32 and the RealSense are used -->
+      <xacro:if value="${use_realsense}">
+        <!-- Add only the Microstrain 3DM-GX4-45 model for now -->
+        <!-- TODO make the xacro parametric against the IMU model -->
+        <xacro:microstrain_gx4_45 parent="frontier_mount" simulation="${simulation}">
+          <!-- the origin is the same for both versions because it's in the -->
+          <!-- middle of the screw holes at the bottom -->
+          <origin xyz="34.047e-3 -34.58733e-3 65.7e-3" rpy="${pi} 0.0 0.0"/>
+        </xacro:microstrain_gx4_45>
+      </xacro:if>
     </xacro:unless>
-    <!-- if it's a model with Hesai PandarXT -->
-    <xacro:if value="${hesai}">
-      <xacro:hesai_device name="pandar" parent="frontier_mount" simulation="${simulation}">
-        <!-- 4 mm standoff present, not shown in model -->
-        <origin xyz="0 0 81.7e-3" rpy="0 0 0" />
-      </xacro:hesai_device>
+    <!-- Assuming we are using RealSense D435i -->
+    <xacro:if value="${use_realsense}">
+      <xacro:sensor_d435i name="camera" parent="realsense_parent" use_nominal_extrinsics="${simulation}">
+        <origin xyz="0 0 0" rpy="0 0 0" />
+      </xacro:sensor_d435i>
+      <link name="realsense_parent" />
+      <joint name="base_to_realsense" type="fixed">
+        <origin xyz="73.65e-3 7.5e-3 50.75e-3" rpy="0 0 0" />
+        <parent link="frontier_mount" />
+        <child link="realsense_parent" />
+      </joint>
     </xacro:if>
-    <!-- add RealSense D435i (the mesh is actually the non-IMU version) -->
-    <xacro:sensor_d435i name="camera" parent="realsense_parent" use_nominal_extrinsics="${simulation}">
-      <origin xyz="0 0 0" rpy="0 0 0" />
-    </xacro:sensor_d435i>
-    <link name="realsense_parent" />
-    <joint name="base_to_realsense" type="fixed">
-      <origin xyz="73.65e-3 7.5e-3 50.75e-3" rpy="0 0 0" />
-      <parent link="frontier_mount" />
-      <child link="realsense_parent" />
-    </joint>
-    <!-- Add the Microstrain 3DM-GX4-45 for now -->
-    <!-- TODO make the xacro parametric against the IMU model -->
-    <xacro:microstrain_gx4_45 parent="frontier_mount" simulation="${simulation}">
-      <!-- the origin is the same for both versions because it's in the -->
-      <!-- middle of the screw holes at the bottom -->
-      <origin xyz="34.047e-3 -34.58733e-3 65.7e-3" rpy="${pi} 0.0 0.0"/>
-    </xacro:microstrain_gx4_45>
+    <!-- Assuming we are using Alphasense Core Dev Kit -->
+    <xacro:unless value="${use_realsense}">
+        <xacro:alphasense parent="frontier_mount" four_cams="true">
+          <origin xyz="32e-3 0.0 47.7e-3" rpy="0 0 0" />
+        </xacro:alphasense>
+    </xacro:unless>
     <!-- the geometric center of the bottom screws is not
          perfectly coincident with the base frame

File: urdf/frontier_standalone.urdf.xacro (robot description, xacro)
@@ -14,8 +14,20 @@
   <xacro:include filename="$(find frontier_description)/urdf/frontier.urdf.xacro" />
   <xacro:arg name="simulation" default="false" />
-  <!-- Need to put the arithmetic computation into quotes because args must be strings -->
-  <xacro:arg name="ouster_rotation" default="'${-pi/4}'" />
+  <!-- If true, use Ouster OS1-64. If false, use HESAI XT32 -->
+  <xacro:arg name="use_ouster" default="false" />
+  <!-- If true, use RealSense d435i. Otherwise, use Alphasense Core -->
+  <xacro:arg name="use_realsense" default="false" />
+  <!-- If true, rotate the Ouster by 45 deg. Otherwise keep zero.
+       If use_ouster is false, the argument is ignored -->
+  <xacro:arg name="rotate_ouster" default="false" />
+  <!-- If true, raise the lidar by 4mm.
+       If use_realsense is false, the argument is ignored -->
+  <xacro:arg name="raise_lidar" default="false" />
   <link name="base"/>
-  <xacro:frontier_device parent="base" simulation="$(arg simulation)" ouster_rotation="$(arg ouster_rotation)">
+  <xacro:frontier_device parent="base" simulation="$(arg simulation)"
+                         use_ouster="$(arg use_ouster)"
+                         use_realsense="$(arg use_realsense)"
+                         rotate_ouster="$(arg rotate_ouster)"
+                         raise_lidar="$(arg raise_lidar)">
     <!-- this transform makes the robot base coincident with the front camera link -->
     <origin xyz="-0.08425 -0.025 -0.06325" rpy="0 0 0" />

Commit message: Add hesai (#13)
* add option to load hesai

* fix microstrain

* remove old stuff from rviz config

* remove ground camera and other old names

* add mesh for gx4_25 IMU

* move microstrains to dedicated file, load the 45 one into the xacro

* create unique frontier device

* fix missing package dependencies

File: urdf/frontier.urdf.xacro (robot description, xacro)
@@ -1,4 +1,4 @@
 <?xml version="1.0"?>
-<!-- Copyright 2020 University of Oxford
+<!-- Copyright 2020-2022 University of Oxford
    Licensed under the Apache License, Version 2.0 (the "License");
    you may not use this file except in compliance with the License.
@@ -15,34 +15,79 @@
   <xacro:include filename="$(find realsense2_description)/urdf/_d435i.urdf.xacro" />
   <xacro:include filename="$(find ouster_description)/urdf/ouster.urdf.xacro" />
+  <xacro:include filename="$(find hesai_description)/urdf/hesai.urdf.xacro" />
+  <xacro:include filename="$(find frontier_description)/urdf/microstrain.urdf.xacro" />
+  <xacro:include filename="$(find alphasense_description)/urdf/alphasense.urdf.xacro" />
   <xacro:macro name="frontier_device" params="parent:=base
                                              *origin
                                              simulation:=false
-                                             ground_camera:=false
-                                             ouster_vertical_angle:=45
-                                             ouster_beams:=64
-                                             ouster_hz:=10
-                                             ouster_rotation:=${-pi/4}">
-    <!-- TODO make the xacro parametric against frontier version -->
-    <link name="frontier_mount">
-      <visual>
-        <origin xyz="0 0 0" rpy="0 0 0" />
-        <geometry>
-          <mesh filename="package://frontier_description/urdf/meshes/frontier_mount_v3.dae" />
-        </geometry>
-      </visual>
-      <inertial>
-        <!-- TODO Update inertia parameters -->
-        <origin xyz="-12.256e-3 -0.092e-3 -29.959e-3" rpy="0 0 0" />
-        <mass value="0.212" />
-        <inertia ixx="3.541e-4" ixy="5.656e-6" ixz="-6.046e-5"
-                 iyy="5.340e-4" iyz="-7.84e-6" izz="3.672e-4" />
-        </inertial>
-        <collision>
-	  <origin xyz="7e-3 0 ${77.25e-3/2}" rpy="0 0 0" />
+                                             use_ouster:=false
+                                             use_realsense:=false
+                                             rotate_ouster:=false
+                                             raise_lidar:=false">
+    <xacro:property name="lidar_hz" value="10" />
+    <xacro:if value="${use_realsense}">
+      <xacro:if value="${raise_lidar}">
+        <!-- 4 mm standoff present, not shown in model -->
+        <xacro:property name="lidar_z" value="81.7e-3"/>
+      </xacro:if>
+      <xacro:unless value="${raise_lidar}">
+        <xacro:property name="lidar_z" value="77.7e-3"/>
+      </xacro:unless>
+    </xacro:if>
+    <xacro:unless value="${use_realsense}">
+      <!-- lidar is 1 mm higher than in the previous version of the halo -->
+      <xacro:property name="lidar_z" value="91.683e-3"/>
+    </xacro:unless>
+    <!-- Assuming we are using Ouster OS1-64 -->
+    <xacro:if value="${use_ouster}">
+      <xacro:property name="lidar_fov" value="45" />
+      <xacro:property name="lidar_beams" value="64"/>
+    </xacro:if>
+    <!-- assuming we are using Hesai XT32 -->
+    <xacro:unless value="${use_ouster}">
+      <xacro:property name="lidar_fov" value="31" />
+      <xacro:property name="lidar_beams" value="32"/>
+    </xacro:unless>
+    <xacro:if value="${rotate_ouster}">
+      <xacro:property name="ouster_rotation" value="${-pi/4}"/>
+    </xacro:if>
+    <xacro:unless value="${rotate_ouster}">
+      <xacro:property name="ouster_rotation" value="0"/>
+    </xacro:unless>
+    <!-- Assuming we are using RealSense D435i -->
+    <xacro:if value="${use_realsense}">
+      <link name="frontier_mount">
+        <visual>
+          <origin xyz="0.0 0.0 0.0" rpy="0.0 0.0 0.0" />
           <geometry>
-            <box size="133e-3 114e-3 77.25e-3" />
+            <mesh filename="package://frontier_description/urdf/meshes/frontier_mount_v6_realsense.dae" />
           </geometry>
-        </collision>
-    </link>
+        </visual>
+        <inertial>
+          <!-- TODO Update inertia parameters -->
+          <origin xyz="-12.256e-3 -0.092e-3 -29.959e-3" rpy="0 0 0" />
+          <mass value="0.212" />
+          <inertia ixx="3.541e-4" ixy="5.656e-6" ixz="-6.046e-5"
+                   iyy="5.340e-4" iyz="-7.84e-6" izz="3.672e-4" />
+          </inertial>
+          <collision>
+	    <origin xyz="7e-3 0 ${77.25e-3/2}" rpy="0 0 0" />
+            <geometry>
+              <box size="133e-3 114e-3 77.25e-3" />
+            </geometry>
+          </collision>
+      </link>
+    </xacro:if>
+    <!-- Assuming we are using Alphasense Core Dev Kit -->
+    <xacro:unless value="${use_realsense}">
+      <link name="frontier_mount">
+        <visual>
+          <geometry>
+            <mesh filename="package://frontier_description/urdf/meshes/frontier_mount_v6.dae" />
+          </geometry>
+        </visual>
+        <!-- TODO add inertia params -->
+      </link>
+    </xacro:unless>
     <joint name="${parent}_to_mount" type="fixed">
       <parent link="${parent}" />
@@ -50,22 +95,49 @@
       <xacro:insert_block name="origin" />
     </joint>
-    <!-- add OS Ouster Lidar sensor -->
-    <xacro:os_device name="os1_sensor" parent="frontier_mount" simulation="${simulation}">
-      <origin xyz="0 0 77.258e-3" rpy="0 0 ${ouster_rotation}" />
-    </xacro:os_device>
-    <!-- add RealSense D435i (the mesh is actually the non-IMU version -->
-    <xacro:sensor_d435i name="camera" parent="realsense_parent" use_nominal_extrinsics="${simulation}">
-      <origin xyz="0 0 0" rpy="0 0 0" />
-    </xacro:sensor_d435i>
-    <link name="realsense_parent" />
-    <joint name="base_to_realsense" type="fixed">
-      <origin xyz="73.65e-3 7.5e-3 50.75e-3" rpy="0 0 0" />
-      <parent link="frontier_mount" />
-      <child link="realsense_parent" />
-    </joint>
+    <!-- Assuming we are using Ouster OS1-64 -->
+    <xacro:if value="${use_ouster}">
+      <!-- add OS Ouster Lidar sensor -->
+      <xacro:os_device name="os_sensor" parent="frontier_mount" simulation="${simulation}">
+        <origin xyz="0 0 ${lidar_z}" rpy="0 0 ${ouster_rotation}" />
+      </xacro:os_device>
+    </xacro:if>
+    <!-- assuming we are using Hesai XT32 -->
+    <xacro:unless value="${use_ouster}">
+      <xacro:hesai_device name="pandar" parent="frontier_mount" simulation="${simulation}">
+          <origin xyz="0 0 ${lidar_z}" rpy="0 0 0" />
+      </xacro:hesai_device>
+      <!-- Only add the Microstrain if the Hesai XT32 and the RealSense are used -->
+      <xacro:if value="${use_realsense}">
+        <!-- Add only the Microstrain 3DM-GX4-45 model for now -->
+        <!-- TODO make the xacro parametric against the IMU model -->
+        <xacro:microstrain_gx4_45 parent="frontier_mount" simulation="${simulation}">
+          <!-- the origin is the same for both versions because it's in the -->
+          <!-- middle of the screw holes at the bottom -->
+          <origin xyz="34.047e-3 -34.58733e-3 65.7e-3" rpy="${pi} 0.0 0.0"/>
+        </xacro:microstrain_gx4_45>
+      </xacro:if>
+    </xacro:unless>
+    <!-- Assuming we are using RealSense D435i -->
+    <xacro:if value="${use_realsense}">
+      <xacro:sensor_d435i name="camera" parent="realsense_parent" use_nominal_extrinsics="${simulation}">
+        <origin xyz="0 0 0" rpy="0 0 0" />
+      </xacro:sensor_d435i>
+      <link name="realsense_parent" />
+      <joint name="base_to_realsense" type="fixed">
+        <origin xyz="73.65e-3 7.5e-3 50.75e-3" rpy="0 0 0" />
+        <parent link="frontier_mount" />
+        <child link="realsense_parent" />
+      </joint>
+    </xacro:if>
+    <!-- Assuming we are using Alphasense Core Dev Kit -->
+    <xacro:unless value="${use_realsense}">
+        <xacro:alphasense parent="frontier_mount" four_cams="true">
+          <origin xyz="32e-3 0.0 47.7e-3" rpy="0 0 0" />
+        </xacro:alphasense>
+    </xacro:unless>
     <!-- the geometric center of the bottom screws is not
          perfectly coincident with the base frame
          (i.e., geometry center of device,
-         coincident with ouster center) -->
+         coincident with lidar's rotation center) -->
     <link name="bottom_screws_center" />
     <joint name="frontier_mount_to_bottom_screws_center" type="fixed">
@@ -74,36 +146,12 @@
       <child link="bottom_screws_center" />
     </joint>
-    <xacro:if value="${ground_camera}">
-      <link name="ground_camera_shim">
-        <visual>
-          <geometry>
-            <mesh filename="package://frontier_description/urdf/meshes/frontier_40deg_shim.dae" />
-          </geometry>
-        </visual>
-        <inertial>
-        <!-- TODO Update inertia parameters -->
-        <origin xyz="9.513e-3 -2.85e-3 -12.423e-3" rpy="0 0 0" />
-        <mass value="0.01" />
-        <inertia ixx="10.931e-6" ixy="0.177e-6" ixz="-0.253e-6"
-                 iyy="1.199e-6" iyz="0.075e-6" izz="10.21e-6" />
-        </inertial>
-      </link>
-      <joint name="ground_camera_shim_joint" type="fixed">
-        <origin xyz="59.5e-3 0 38.7e-3" rpy="0 0 0" />
-        <parent link="frontier_mount" />
-        <child link="ground_camera_shim" />
-      </joint>
-      <xacro:sensor_d435i name="ground_camera" parent="ground_camera_shim" use_nominal_extrinsics="${simulation}">
-        <origin xyz="14.345e-3 7.5e-3 -25.212e-3" rpy="0 ${pi*40.0/180.0} 0" />
-      </xacro:sensor_d435i>
-    </xacro:if>
     <!-- Bring in simulation data for Gazebo. -->
     <xacro:if value="${simulation}">
       <!-- Simulated Ouster -->
       <xacro:include filename="$(find frontier_description)/urdf/gazebo/ouster.gazebo"/>
-      <xacro:ouster_gazebo name="ouster" min_vertical_angle="${ouster_vertical_angle}"
-                                         max_vertical_angle="${-ouster_vertical_angle}"
-                                         hz="${ouster_hz}"
-                                         lasers="${ouster_beams}">
+      <xacro:ouster_gazebo name="ouster" min_vertical_angle="${lidar_fov}"
+                                         max_vertical_angle="${-lidar_fov}"
+                                         hz="${lidar_hz}"
+                                         lasers="${lidar_beams}">
         <origin xyz="0 0 0" rpy="0 0 0" />
       </xacro:ouster_gazebo>
@@ -114,10 +162,4 @@
         <origin xyz="0 0 0" rpy="0 0 0"/>
       </xacro:realsense_d435_gazebo>
-      <!-- Add ground camera -->
-      <xacro:if value="${ground_camera}">
-        <xacro:realsense_d435_gazebo name="ground_camera">
-          <origin xyz="0 0 0" rpy="0 0 0"/>
-        </xacro:realsense_d435_gazebo>
-      </xacro:if>
       <!-- Add ground truth -->
       <xacro:include filename="$(find frontier_description)/urdf/gazebo/ground_truth.gazebo"/>

File: urdf/frontier_standalone.urdf.xacro (robot description, xacro)
@@ -14,9 +14,20 @@
   <xacro:include filename="$(find frontier_description)/urdf/frontier.urdf.xacro" />
   <xacro:arg name="simulation" default="false" />
-  <xacro:arg name="ground_camera" default="false" />
-  <!-- Need to put the arithmetic computation into quotes because args must be strings -->
-  <xacro:arg name="ouster_rotation" default="'${-pi/4}'" />
+  <!-- If true, use Ouster OS1-64. If false, use HESAI XT32 -->
+  <xacro:arg name="use_ouster" default="false" />
+  <!-- If true, use RealSense d435i. Otherwise, use Alphasense Core -->
+  <xacro:arg name="use_realsense" default="false" />
+  <!-- If true, rotate the Ouster by 45 deg. Otherwise keep zero.
+       If use_ouster is false, the argument is ignored -->
+  <xacro:arg name="rotate_ouster" default="false" />
+  <!-- If true, raise the lidar by 4mm.
+       If use_realsense is false, the argument is ignored -->
+  <xacro:arg name="raise_lidar" default="false" />
   <link name="base"/>
-  <xacro:frontier_device parent="base" simulation="$(arg simulation)" ground_camera="$(arg ground_camera)" ouster_rotation="$(arg ouster_rotation)">
+  <xacro:frontier_device parent="base" simulation="$(arg simulation)"
+                         use_ouster="$(arg use_ouster)"
+                         use_realsense="$(arg use_realsense)"
+                         rotate_ouster="$(arg rotate_ouster)"
+                         raise_lidar="$(arg raise_lidar)">
     <!-- this transform makes the robot base coincident with the front camera link -->
     <origin xyz="-0.08425 -0.025 -0.06325" rpy="0 0 0" />
