Commit message: update for frontier frn-0007

File: urdf/frontier.urdf.xacro (robot description, xacro)
@@ -29,8 +29,8 @@
       <xacro:if value="${raise_lidar}">
         <!-- 4 mm standoff present, not shown in model -->
-        <xacro:property name="lidar_z" value="81.7e-3"/>
+        <xacro:property name="lidar_z" value="77e-3"/>
       </xacro:if>
       <xacro:unless value="${raise_lidar}">
-        <xacro:property name="lidar_z" value="77.7e-3"/>
+        <xacro:property name="lidar_z" value="73e-3"/>
       </xacro:unless>
     </xacro:if>
